Commit message: Fix robot stability with front/back caster wheels

File: urdf/robot.urdf (robot description, URDF)
Before this commit: robot my_robot, 3 links, 2 joints
Links:
- added link back_caster, mass 0.05; collision sphere radius=0.02; visual sphere radius=0.02
- added link front_caster, mass 0.05; collision sphere radius=0.02; visual sphere radius=0.02
Joints:
- added joint back_caster_joint: type fixed, parent base_link, child back_caster, origin xyz=-0.12 0.0 -0.055 rpy=0 0 0
- added joint front_caster_joint: type fixed, parent base_link, child front_caster, origin xyz=0.12 0.0 -0.055 rpy=0 0 0
