Commit message: Phase 5: Add lidar sensor to URDF

File: my_robot/urdf/robot.urdf (robot description, URDF)
Before this commit: robot my_robot, 5 links, 4 joints
Links:
- added link lidar_link, mass 0.05; collision cylinder length=0.04 radius=0.03; visual cylinder length=0.04 radius=0.03
Joints:
- added joint lidar_joint: type fixed, parent base_link, child lidar_link, origin xyz=0.0 0.0 0.07 rpy=0 0 0

Commit message: Redesign robot as forklift, integrate AWS warehouse world for pallet-avoidance project

File: my_robot/urdf/robot.urdf (robot description, URDF)
Before this commit: robot my_robot, 6 links, 5 joints
Links:
- added link left_fork, mass 0.05; collision box size=0.35 0.04 0.02; visual box size=0.35 0.04 0.02
- added link mast, mass 0.1; collision box size=0.05 0.18 0.35; visual box size=0.05 0.18 0.35
- added link right_fork, mass 0.05; collision box size=0.35 0.04 0.02; visual box size=0.35 0.04 0.02
Joints:
- added joint left_fork_joint: type fixed, parent base_link, child left_fork, origin xyz=0.325 0.06 -0.06 rpy=0 0 0
- added joint mast_joint: type fixed, parent base_link, child mast, origin xyz=0.16 0.0 0.225 rpy=0 0 0
- added joint right_fork_joint: type fixed, parent base_link, child right_fork, origin xyz=0.325 -0.06 -0.06 rpy=0 0 0

Commit message: Phase 7a: OpenCV-based pallet detection, verified against captured warehouse imagery

File: my_robot/urdf/robot.urdf (robot description, URDF)
Before this commit: robot my_robot, 9 links, 8 joints
Links:
- added link camera_link, mass 0.02; collision box size=0.03 0.03 0.03; visual box size=0.03 0.03 0.03
Joints:
- added joint camera_joint: type fixed, parent base_link, child camera_link, origin xyz=0.19 0.0 0.4 rpy=0 0 0

Commit message: Phase 7: Working ROS2 action server for autonomous navigation, fixed lidar self-detection bug from mast geometry

File: my_robot/urdf/robot.urdf (robot description, URDF)
Before this commit: robot my_robot, 10 links, 9 joints
Joints:
- joint lidar_joint: origin xyz=0.0 0.0 0.07 rpy=0 0 0 -> xyz=0.0 0.0 0.45 rpy=0 0 0

Commit message: Scale up forklift 3x for environment fit, implement bug-algorithm style obstacle avoidance (turn-step-recheck logic)

File: my_robot/urdf/robot.urdf (robot description, URDF)
Before this commit: robot my_robot, 10 links, 9 joints
Links:
- link back_caster: mass 0.05 -> 0.15; geometry collision sphere radius=0.06; visual sphere radius=0.06
- link base_link: mass 1.0 -> 3.0; geometry collision box size=0.9 0.6 0.3; visual box size=0.9 0.6 0.3
- link camera_link: mass 0.02 -> 0.06; geometry collision box size=0.09 0.09 0.09; visual box size=0.09 0.09 0.09
- link front_caster: mass 0.05 -> 0.15; geometry collision sphere radius=0.06; visual sphere radius=0.06
- link left_fork: mass 0.05 -> 0.15; geometry collision box size=1.05 0.12 0.06; visual box size=1.05 0.12 0.06
- link left_wheel: mass 0.1 -> 0.3; geometry collision cylinder length=0.12 radius=0.15; visual cylinder length=0.12 radius=0.15
- link lidar_link: mass 0.05 -> 0.15; geometry collision cylinder length=0.12 radius=0.09; visual cylinder length=0.12 radius=0.09
- link mast: mass 0.1 -> 0.3; geometry collision box size=0.15 0.54 1.05; visual box size=0.15 0.54 1.05
- link right_fork: mass 0.05 -> 0.15; geometry collision box size=1.05 0.12 0.06; visual box size=1.05 0.12 0.06
- link right_wheel: mass 0.1 -> 0.3; geometry collision cylinder length=0.12 radius=0.15; visual cylinder length=0.12 radius=0.15
Joints:
- joint back_caster_joint: origin xyz=-0.12 0.0 -0.055 rpy=0 0 0 -> xyz=-0.36 0.0 -0.2 rpy=0 0 0
- joint camera_joint: origin xyz=0.19 0.0 0.4 rpy=0 0 0 -> xyz=0.57 0.0 1.2 rpy=0 0 0
- joint front_caster_joint: origin xyz=0.12 0.0 -0.055 rpy=0 0 0 -> xyz=0.36 0.0 -0.2 rpy=0 0 0
- joint left_fork_joint: origin xyz=0.325 0.06 -0.06 rpy=0 0 0 -> xyz=0.975 0.18 -0.18 rpy=0 0 0
- joint left_wheel_joint: origin xyz=0.0 0.12 -0.025 rpy=-1.5708 0 0 -> xyz=0.0 0.36 -0.075 rpy=-1.5708 0 0
- joint lidar_joint: origin xyz=0.0 0.0 0.45 rpy=0 0 0 -> xyz=0.0 0.0 1.35 rpy=0 0 0
- joint mast_joint: origin xyz=0.16 0.0 0.225 rpy=0 0 0 -> xyz=0.48 0.0 0.675 rpy=0 0 0
- joint right_fork_joint: origin xyz=0.325 -0.06 -0.06 rpy=0 0 0 -> xyz=0.975 -0.18 -0.18 rpy=0 0 0
- joint right_wheel_joint: origin xyz=0.0 -0.12 -0.025 rpy=-1.5708 0 0 -> xyz=0.0 -0.36 -0.075 rpy=-1.5708 0 0
